File: hardware/discrete fan controller.brd (EAGLE design)
At the start: 22 x 15.2 mm, 13 parts, among them Q1 BCX56, U1 TL431

Commit message: TL431 Minimum current
4K7 changed to 1K.
Parts:
- R1: value 4K7 -> 1K
Changed lines of the file:
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@@
 <attribute name="VALUE" x="9.4085" y="5.922" size="0.6096" layer="27" font="vector" ratio="15" rot="R270"/>
 </element>
-<element name="R1" library="ipc-7351-resistor" package="RESC1608X55N" value="4K7" x="12.573" y="3.429" smashed="yes" rot="R270">
+<element name="R1" library="ipc-7351-resistor" package="RESC1608X55N" value="1K" x="12.573" y="3.429" smashed="yes" rot="R270">
 <attribute name="NAME" x="12.212" y="5.1355" size="0.6096" layer="25" font="vector" ratio="15"/>
 <attribute name="VALUE" x="12.2635" y="4.044" size="0.6096" layer="27" font="vector" ratio="15" rot="R270"/>
